File: RaspiCar-Interface-Board/RasPiCar-KiCAD-v1.2/RasPi-Car.kicad_pcb (KiCad board)
At the start: 2 copper layers, 108.7 x 63.5 mm, 71 parts, among them J1 PowerSupply, J10 Ser, J2 Raspi, J3 Motor Left, J4 Motor Right, J5 SPI, J6 LiDAR, J7 LCD, J8 I2C, J9 Vcc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

Commit message: Bug fixes
Parts:
- Q2: value IRLML6401 -> IRLML2244
Changed lines of the file:
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@@
         (effects (font (size 1 1) (thickness 0.15)))
     )
-    (fp_text value "IRLML6401" (at 0 2.4) (layer "F.SilkS")
+    (fp_text value "IRLML2244" (at 0 2.4) (layer "F.SilkS")
         (effects (font (size 1 1) (thickness 0.15)))
     )
