File: RaspiCar-Interface-Board/RasPiCar-KiCAD-v1.2/RasPi-Car.kicad_sch (KiCad schematic)
At the start: 69 parts, among them J1 PowerSupply, J10 Ser, J2 Raspi, J3 Motor Left, J4 Motor Right, J5 SPI, J6 LiDAR, J7 LCD, J8 I2C, J9 Vcc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

Commit message: Bug fixes
Parts:
- Q2: value IRLML6401 -> IRLML2244
Changed lines of the file:
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@@
       (effects (font (size 1.27 1.27)))
     )
-    (property "Value" "IRLML6401" (at 217.805 52.6796 90)
+    (property "Value" "IRLML2244" (at 217.805 52.6796 90)
       (effects (font (size 1.27 1.27)))
     )
